File: boards/lin_node_v1/lin_node.sch (EAGLE design)
At the start: 27 parts, among them J1 AVR_SPI_PRG_6NS, U1 ATtiny167, U2 MCP2025, U3 VNQ5160K

Commit message: Update to current sample boards
Parts:
- removed +12V, OUT1, OUT2, OUT3, OUT4: WIREPADTH-2.0MM, custom:WIREPADTH-2.0MM
- removed D2: 1N4004, custom:1N4004
- removed GND, LIN: WIREPAD2,54/1,0, custom:WIREPAD2,54/1,0
- removed RN2, RN3: 10K, custom:E4RP
- removed RN4, RN5: 10K, custom:G04R
- removed U3: VNQ5160K, custom:VNQ5160K
- added SV1: (no value), custom:FE08-2
- added U$1, U$2: MOUNT-HOLE3.1MM, custom:MOUNT-HOLE3.1MM
Connections:
- removed net N$1: D4.C, LIN.P, U2.LIN
- removed net N$10: RN3A.2, RN4.2, U3.STATUS1
- removed net N$11: RN2A.2, U3.INPUT1
- removed net N$12: RN2D.2, U3.INPUT4
- removed net N$13: RN2C.2, U3.INPUT3
- removed net N$14: RN2B.2, U3.INPUT2
- removed net N$6: RN3D.2, RN4.3, U3.STATUS4
- removed net N$7: RN3C.2, RN4.4, U3.STATUS3
- removed net N$8: D2.A, RN1C.2, U3.GND, U3.STAT_DIS
- removed net N$9: RN3B.2, RN4.5, U3.STATUS2
- removed net OUT1: RN2A.1, U1.(PCINT8/OC1AU/DI/SDA)PB0
- removed net OUT2: RN2B.1, U1.(PCINT10/OC1AV/USCK/SCL)PB2
- removed net OUT3: RN2C.1, U1.(PCINT12/OC1AW/XTAL1/CLKI)PB4
- removed net OUT4: RN2D.1, U1.(PCINT14/ADC9/OC1AX/INT0)PB6
- removed net OUTPUT1: OUT1.P, RN5.2, U3.OUTPUT1A, U3.OUTPUT1B, U3.OUTPUT1C
- removed net OUTPUT2: OUT2.P, RN5.3, U3.OUTPUT2A, U3.OUTPUT2B, U3.OUTPUT2C
- removed net OUTPUT3: OUT3.P, RN5.4, U3.OUTPUT3A, U3.OUTPUT3B, U3.OUTPUT3C
- removed net OUTPUT4: OUT4.P, RN5.5, U3.OUTPUT4A, U3.OUTPUT4B, U3.OUTPUT4C
- removed net STATUS1: RN3A.1, U1.(PCINT9/AC1BU/DO)PB1
- removed net STATUS2: RN3B.1, U1.(PCINT11/OC1BV)PB3
- removed net STATUS3: RN3C.1, U1.(PCINT13/ADC8/OC1BW/XTAL2/CLKO)PB5
- removed net STATUS4: RN3D.1, U1.PA7(AREF/XREF/AIN1/ADC7/PCINT7)
- new net LIN: D4.C, SV1.6, U2.LIN
- new net P0/SDA: SV1.1, U1.(PCINT8/OC1AU/DI/SDA)PB0
- new net P1: SV1.3, U1.(PCINT9/AC1BU/DO)PB1
- new net P2/SCL: SV1.5, U1.(PCINT10/OC1AV/USCK/SCL)PB2
- new net P3: SV1.7, U1.(PCINT11/OC1BV)PB3
- new net P4: SV1.9, U1.(PCINT12/OC1AW/XTAL1/CLKI)PB4
- new net P5/ADC8: SV1.11, U1.(PCINT13/ADC8/OC1BW/XTAL2/CLKO)PB5
- new net P6/ADC9: SV1.13, U1.(PCINT14/ADC9/OC1AX/INT0)PB6
- new net P7/ADC7: SV1.15, U1.PA7(AREF/XREF/AIN1/ADC7/PCINT7)
- net +12V: now also SV1.2; no longer +12V.P, U3.VCC1, U3.VCC12, U3.VCC_TAB
- net +5V: now also SV1.4; no longer RN4.1, RN5.1
- net GND: now also SV1.10, SV1.8; no longer D2.C, GND.P
- net MISO: now also SV1.12
- net MOSI: now also SV1.14
- net SCK: now also SV1.16
Other:
- moved on the sheet: C1, C2, C3, D1, D3, D4, F1, J1, LED1, LED2, RN1A, RN1B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
